File: Zocalo-mcp2515.sch (EAGLE design)
At the start: 0 parts

Commit message: fix
Parts:
- added IC1: (no value), can:MCP2515SO
- added JP1, JP2: (no value), pinhead:PINHD-1X9
Connections:
- new net GND: JP1.9
- new net N$1: IC1D.TXCAN, JP1.1
- new net N$10: IC1D.RX0BF, JP2.8
- new net N$11: IC1D.INT, JP2.7
- new net N$12: IC1D.SCK, JP2.6
- new net N$13: IC1D.SI, JP2.5
- new net N$14: IC1D.SO, JP2.4
- new net N$15: IC1D.CS, JP2.3
- new net N$16: IC1D.RESET, JP2.2
- new net N$2: IC1D.RXCAN, JP1.2
- new net N$3: IC1D.TX0RTS, JP1.4
- new net N$4: IC1D.TX1RTS, JP1.5
- new net N$5: IC1D.TX2RTS, JP1.6
- new net N$6: IC1D.CLKOUT, JP1.3
- new net N$7: IC1D.OSC2, JP1.7
- new net N$8: IC1D.OSC1, JP1.8
- new net N$9: IC1D.RX1BF, JP2.9
- new net VCC: JP2.1
